Commit message: visual odometry + saliency

File: mighty_rover/xacro/diff_drive.xacro (robot description, xacro)
@@ -176,47 +176,4 @@
       </sensor>
     </gazebo>
-<!--<link name="hokuyo_sensor">
-  <visual>
-    <origin xyz="0 0 0" rpy="0 0 0"/>
-   <geometry>
-     <box size="0.05 0.05 0.05"/>
-   </geometry>
-   <material name="Blue"/>
-   </visual>
- </link>
-<joint name="hokuyo_joint" type="fixed">
-  <origin xyz="0.07 0 0.08" rpy="0 0 0"/>
-  <parent link="base_link"/>
-  <child link="hokuyo_sensor"/>
-</joint>
-<gazebo reference="hokuyo_sensor">
-  <material>Gazebo/Blue</material>
-  <turnGravityOff>false</turnGravityOff>
-  <sensor type="ray" name="base_link_hokuyo_sensor">
-   <pose>0.025 0 0 0 0 0</pose>
-   <visualize>false</visualize>
-   <update_rate>40</update_rate>
-   <ray>
-     <scan>
-       <horizontal>
-         <samples>720</samples>
-         <resolution>1</resolution>
-         <min_angle>-1.57</min_angle>
-         <max_angle>1.57</max_angle>
-        </horizontal>
-      </scan>
-     <range>
-        <min>0.10</min>
-        <max>10.0</max>
-        <resolution>0.001</resolution>
-      </range>
-     </ray>
-     <plugin name="gazebo_ros_head_hokuyo_controller"
-          filename="libgazebo_ros_laser.so">
-        <topicName>/scan</topicName>
-        <frameName>hokuyo_sensor</frameName>
-       </plugin>
-      </sensor>
-     </gazebo>   -->
 <link name="hokuyo_sensor">
 <collision>
@@ -246,5 +203,5 @@
     <sensor type="gpu_ray" name="base_link_hokuyo_sensor">
       <pose>0 0 0 0 0 0</pose>
-      <visualize>true</visualize>
+      <visualize>false</visualize>
       <update_rate>40</update_rate>
       <ray>
@@ -297,5 +254,5 @@
   </link>
   <joint name="camera_joint" type="fixed">
-    <origin xyz="0 0 0" rpy="0 0 ${M_PI/2}"/>
+    <origin xyz="0 0 0" rpy="${M_PI/-2} 0 ${M_PI/-2}"/>
     <parent link="base_link"/>
     <child link="camera_link"/>
@@ -308,4 +265,5 @@
         <camera>
           <horizontal_fov>${60.0*M_PI/180.0}</horizontal_fov>
+          <pose>0 0 0 0 ${radians(-90)} ${radians(90)}</pose>
           <image>
             <format>B8G8R8</format>

File: mighty_rover/xacro/mighty.xacro (robot description, xacro)
@@ -136,7 +136,4 @@
   <dynamics damping="0.0" friction="0.0"/>
 </joint>
---
---
---
  <transmission name="${prefix}_${suffix}_wheel_trans">
       <type>transmission_interface/SimpleTransmission</type>
@@ -150,9 +147,4 @@
  </transmission>
 </xacro:macro>
-<!--<xacro:macro name="body"parent="base_link" />
-<xacro:wheel prefix="right" suffix="front" parent="base_link" X="1" Y="0" Z="-1"/>
-<xacro:wheel prefix="right" suffix="back" parent="base_link" X="0" Y="1" Z="-1"/>
-<xacro:wheel prefix="left" suffix="front" parent="base_link" X="1" Y="0" Z="1"/>
-<xacro:wheel prefix="left" suffix="back" parent="base_link" X="0" Y="1" Z="1"/>-->
 <xacro:wheel prefix="right" suffix="front" X="1" Y="0" Z="-1"/>
 <xacro:wheel prefix="right" suffix="back" X="0" Y="1" Z="-1"/>
@@ -185,47 +177,4 @@
       </sensor>
     </gazebo>
-<!--<link name="hokuyo_sensor">
-  <visual>
-    <origin xyz="0 0 0" rpy="0 0 0"/>
-   <geometry>
-     <box size="0.05 0.05 0.05"/>
-   </geometry>
-   <material name="Blue"/>
-   </visual>
- </link>
-<joint name="hokuyo_joint" type="fixed">
-  <origin xyz="0.07 0 0.08" rpy="0 0 0"/>
-  <parent link="base_link"/>
-  <child link="hokuyo_sensor"/>
-</joint>
-<gazebo reference="hokuyo_sensor">
-  <material>Gazebo/Blue</material>
-  <turnGravityOff>false</turnGravityOff>
-  <sensor type="ray" name="base_link_hokuyo_sensor">
-   <pose>0.025 0 0 0 0 0</pose>
-   <visualize>false</visualize>
-   <update_rate>40</update_rate>
-   <ray>
-     <scan>
-       <horizontal>
-         <samples>720</samples>
-         <resolution>1</resolution>
-         <min_angle>-1.57</min_angle>
-         <max_angle>1.57</max_angle>
-        </horizontal>
-      </scan>
-     <range>
-        <min>0.10</min>
-        <max>10.0</max>
-        <resolution>0.001</resolution>
-      </range>
-     </ray>
-     <plugin name="gazebo_ros_head_hokuyo_controller"
-          filename="libgazebo_ros_laser.so">
-        <topicName>/scan</topicName>
-        <frameName>hokuyo_sensor</frameName>
-       </plugin>
-      </sensor>
-     </gazebo>   -->
 <link name="hokuyo_sensor">
 <collision>
@@ -264,5 +213,5 @@
               <resolution>1</resolution>
               <min_angle>${radians(-150)}</min_angle>
-              <max_angle>${radians( 150)}</max_angle>-->
+              <max_angle>${radians( 150)}</max_angle>
             <!--<min_angle>-1.570796</min_angle>
             <max_angle>1.570796</max_angle>-->
@@ -285,19 +234,25 @@
     </sensor>
     </gazebo>
-    <property name="M_PI" value="3.14159274"/>
-    <link name="camera_link">
-        <visual>
-        <!--origin xyz="0.05 0 0.05" rpy="0 0 0"/-->
-          <geometry>
-            <mesh filename="package://openni_description/mesh/kinect.dae"/>
-          </geometry>
-        </visual>
-     </link>
-    <joint name="camera_joint" type="fixed">
-      <origin xyz="0.05 0 0.05" rpy="${radians(-90)} 0 ${radians(-90)}"/>
-      <parent link="base_link"/>
-      <child link="camera_link"/>
-    </joint>
-   <gazebo reference="camera_link">
+<property name="M_PI" value="3.14159274"/>
+<link name="camera_link">
+    <visual>
+      <origin xyz="0 0 0" rpy="0 0 0"/>
+      <geometry>
+         <mesh filename="package://openni_description/mesh/kinect.dae"/>
+      </geometry>
+    </visual>
+    <collision>
+        <origin xyz="0.0 0.0 0.0" rpy="0 0 0"/>
+  	    <geometry>
+  	      <box size="0.07271 0.27794 0.073"/>
+  	    </geometry>
+  	  </collision>
+  </link>
+  <joint name="camera_joint" type="fixed">
+    <origin xyz="0 0 0" rpy="0 0 0"/>
+    <parent link="base_link"/>
+    <child link="camera_link"/>
+  </joint>
+<gazebo reference="camera_link">
       <sensor type="depth" name="camera">
         <always_on>true</always_on>
@@ -305,6 +260,6 @@
         <update_rate>20.0</update_rate>
         <camera>
-          <pose>0 0 0 0 ${radians(-90)} ${radians(90)}</pose>
           <horizontal_fov>${60.0*M_PI/180.0}</horizontal_fov>
+          <pose>0 0 0 ${M_PI/2} ${-M_PI/2} 0</pose>
           <image>
             <format>B8G8R8</format>
@@ -337,4 +292,71 @@
       </sensor>
     </gazebo>
+    <!--<property name="M_PI" value="3.14159274"/>
+    <link name="camera_link">
+        <visual>
+        <origin xyz="0.05 0 0.05" rpy="0 0 0"/>
+        </visual>
+     </link>
+    <joint name="camera_joint" type="fixed">
+      <origin xyz="0.05 0 0.05" rpy="0 0 0"/>
+      <parent link="base_link"/>
+      <child link="camera_link"/>
+    </joint>
+   <gazebo reference="camera_link">
+   <sensor type="multicamera" name="stereo_camera">
+      <update_rate>30.0</update_rate>
+      <camera name="left">
+        <pose>0 0.3 0 0 0 0</pose>
+        <horizontal_fov>1.3962634</horizontal_fov>
+        <image>
+          <width>800</width> <!0.7 0.3 0.3 -1.56 -0.78>
+          <height>800</height>
+          <format>R8G8B8</format>
+        </image>
+        <clip>
+          <near>0.02</near>
+          <far>300</far>
+        </clip>
+        <noise>
+          <type>gaussian</type>
+          <mean>0.0</mean>
+          <stddev>0.007</stddev>
+        </noise>
+      </camera>
+      <camera name="right">
+        <pose>0 -0.3 0 0 0 0</pose>
+        <horizontal_fov>1.3962634</horizontal_fov>
+        <image>
+          <width>800</width>
+          <height>800</height>
+          <format>R8G8B8</format>
+        </image>
+        <clip>
+          <near>0.02</near>
+          <far>300</far>
+        </clip>
+        <noise>
+          <type>gaussian</type>
+          <mean>0.0</mean>
+          <stddev>0.007</stddev>
+        </noise>
+      </camera>
+      <plugin name="stereo_camera_controller" filename="libgazebo_ros_multicamera.so">
+        <alwaysOn>true</alwaysOn>
+        <updateRate>30.0</updateRate>
+        <cameraName></cameraName>
+        <imageTopicName>image_raw</imageTopicName>
+        <cameraInfoTopicName>camera_info</cameraInfoTopicName>
+        <frameName>camera_link</frameName>
+        <!<rightFrameName>right_camera_optical_frame</rightFrameName>>
+        <hackBaseline>0.3</hackBaseline>
+        <distortionK1>0.0</distortionK1>
+        <distortionK2>0.0</distortionK2>
+        <distortionK3>0.0</distortionK3>
+        <distortionT1>0.0</distortionT1>
+        <distortionT2>0.0</distortionT2>
+      </plugin>
+    </sensor>
+    </gazebo> -->
 <!-- //////////////////////////////////////////////////////////////// -->
 <!-- ros_control plugin-->

File: mighty_rover/xacro/pf1.xacro (robot description, xacro)
@@ -271,4 +271,56 @@
       </sensor>
     </gazebo>
+        <!-- camera depth joints and links -->
+    <joint name="camera_depth_joint" type="fixed">
+      <origin xyz="0 0 0" rpy="0 0 0"/>
+      <parent link="camera_link"/>
+      <child link="camera_depth_frame" />
+    </joint>
+    <link name="camera_depth_frame"/>
+    <joint name="camera_depth_optical_joint" type="fixed">
+      <origin xyz="0 0 0" rpy="${-M_PI/2} 0 ${-M_PI/2}" />
+      <parent link="camera_depth_frame" />
+      <child link="camera_depth_optical_frame" />
+    </joint>
+    <link name="camera_depth_optical_frame"/>
+    <!-- camera left IR joints and links -->
+    <joint name="camera_left_ir_joint" type="fixed">
+      <origin xyz="0 0 0" rpy="0 0 0" />
+      <parent link="camera_depth_frame" />
+      <child link="camera_left_ir_frame" />
+    </joint>
+    <link name="camera_left_ir_frame"/>
+    <joint name="camera_left_ir_optical_joint" type="fixed">
+      <origin xyz="0 0 0" rpy="${-M_PI/2} 0 ${-M_PI/2}" />
+      <parent link="camera_left_ir_frame" />
+      <child link="camera_left_ir_optical_frame" />
+    </joint>
+    <link name="camera_left_ir_optical_frame"/>
+    <!-- camera right IR joints and links -->
+    <joint name="camera_right_ir_joint" type="fixed">
+      <origin xyz="0 -0.050 0" rpy="0 0 0" />
+      <parent link="camera_depth_frame" />
+      <child link="camera_right_ir_frame" />
+    </joint>
+    <link name="camera_right_ir_frame"/>
+    <joint name="camera_right_ir_optical_joint" type="fixed">
+      <origin xyz="0 0 0" rpy="${-M_PI/2} 0 ${-M_PI/2}" />
+      <parent link="camera_right_ir_frame" />
+      <child link="camera_right_ir_optical_frame" />
+    </joint>
+    <link name="camera_right_ir_optical_frame"/>
+    <!-- camera color joints and links -->
+    <joint name="camera_color_joint" type="fixed">
+      <origin xyz="0 0.015 0" rpy="0 0 0" />
+      <parent link="camera_depth_frame" />
+      <child link="camera_color_frame" />
+    </joint>
+    <link name="camera_color_frame"/>
+    <joint name="camera_color_optical_joint" type="fixed">
+      <origin xyz="0 0 0" rpy="${-M_PI/2} 0 ${-M_PI/2}" />
+      <parent link="camera_color_frame" />
+      <child link="camera_color_optical_frame" />
+    </joint>
+    <link name="camera_color_optical_frame"/>
       <gazebo>
       <plugin name="camera" filename="librealsense_gazebo_plugin.so">
@@ -285,6 +337,6 @@
         <infrared2TopicName>infra2/image_raw</infrared2TopicName>
         <infrared2CameraInfoTopicName>infra2/camera_info</infrared2CameraInfoTopicName>
-        <colorOpticalframeName>color_optical_frame</colorOpticalframeName>
-        <depthOpticalframeName>depth_optical_frame</depthOpticalframeName>
+        <colorOpticalframeName>camera_color_optical_frame</colorOpticalframeName>
+        <depthOpticalframeName>camera_depth_optical_frame</depthOpticalframeName>
         <infrared1OpticalframeName>infrared1_optical_frame</infrared1OpticalframeName>
         <infrared2OpticalframeName>infrared2_optical_frame</infrared2OpticalframeName>
@@ -297,56 +349,4 @@
       </plugin>
     </gazebo>
-    <!-- camera depth joints and links -->
-    <joint name="camera_depth_joint" type="fixed">
-      <origin xyz="0 0 0" rpy="0 0 0"/>
-      <parent link="camera_link"/>
-      <child link="camera_depth_frame" />
-    </joint>
-    <link name="camera_depth_frame"/>
-    <joint name="camera_depth_optical_joint" type="fixed">
-      <origin xyz="0 0 0" rpy="${-M_PI/2} 0 ${-M_PI/2}" />
-      <parent link="camera_depth_frame" />
-      <child link="camera_depth_optical_frame" />
-    </joint>
-    <link name="camera_depth_optical_frame"/>
-    <!-- camera left IR joints and links -->
-    <joint name="camera_left_ir_joint" type="fixed">
-      <origin xyz="0 0 0" rpy="0 0 0" />
-      <parent link="camera_depth_frame" />
-      <child link="camera_left_ir_frame" />
-    </joint>
-    <link name="camera_left_ir_frame"/>
-    <joint name="camera_left_ir_optical_joint" type="fixed">
-      <origin xyz="0 0 0" rpy="${-M_PI/2} 0 ${-M_PI/2}" />
-      <parent link="camera_left_ir_frame" />
-      <child link="camera_left_ir_optical_frame" />
-    </joint>
-    <link name="camera_left_ir_optical_frame"/>
-    <!-- camera right IR joints and links -->
-    <joint name="camera_right_ir_joint" type="fixed">
-      <origin xyz="0 -0.050 0" rpy="0 0 0" />
-      <parent link="camera_depth_frame" />
-      <child link="camera_right_ir_frame" />
-    </joint>
-    <link name="camera_right_ir_frame"/>
-    <joint name="camera_right_ir_optical_joint" type="fixed">
-      <origin xyz="0 0 0" rpy="${-M_PI/2} 0 ${-M_PI/2}" />
-      <parent link="camera_right_ir_frame" />
-      <child link="camera_right_ir_optical_frame" />
-    </joint>
-    <link name="camera_right_ir_optical_frame"/>
-    <!-- camera color joints and links -->
-    <joint name="camera_color_joint" type="fixed">
-      <origin xyz="0 0.015 0" rpy="0 0 0" />
-      <parent link="camera_depth_frame" />
-      <child link="camera_color_frame" />
-    </joint>
-    <link name="camera_color_frame"/>
-    <joint name="camera_color_optical_joint" type="fixed">
-      <origin xyz="0 0 0" rpy="${-M_PI/2} 0 ${-M_PI/2}" />
-      <parent link="camera_color_frame" />
-      <child link="camera_color_optical_frame" />
-    </joint>
-    <link name="camera_color_optical_frame"/>
     <!--end of realsense setup-->
      <link name="hokuyo_sensor">
@@ -1217,7 +1217,7 @@
   <gazebo>
     <plugin name="gazebo_ros_control" filename="libgazebo_ros_control.so">
-      <robotNamespace>/pf1</robotNamespace>
+      <!-- <robotNamespace>/pf1</robotNamespace>
       <robotSimType>gazebo_ros_control/DefaultRobotHWSim</robotSimType>
-      <legacyModeNS>true</legacyModeNS>
+      <legacyModeNS>true</legacyModeNS> -->
       <!-- <commandTopic>cmd_vel</commandTopic>
       <odometryTopic>odom</odometryTopic>
