Commit message: add DEM and waypoint ackermann

File: mighty_rover/xacro/pf1.xacro (robot description, xacro)
@@ -375,5 +375,5 @@
     </joint>
     <gazebo reference="hokuyo_sensor">
-      <sensor type="gpu_ray" name="base_link_hokuyo_sensor">
+      <sensor type="ray" name="base_link_hokuyo_sensor">
         <pose>0 0 0 0 0 0</pose>
         <visualize>false</visualize>
@@ -398,5 +398,5 @@
           </noise>
         </ray>
-        <plugin name="gazebo_ros_lidar_controller" filename="libgazebo_ros_gpu_laser.so">
+        <plugin name="gazebo_ros_lidar_controller" filename="libgazebo_ros_laser.so">
           <topicName>scan</topicName>
           <frameName>hokuyo_sensor</frameName>
@@ -405,5 +405,5 @@
     </gazebo>
     <!-- leg_fl -->
-  <joint name="frame1_fl_to_base_link" type="fixed">
+  <!-- <joint name="frame1_fl_to_base_link" type="fixed">
     <parent link="base_link"/>
     <child  link="frame1_fl"/>
@@ -481,10 +481,10 @@
   <gazebo reference="gear_fl">
     <material>Gazebo/Blue</material>
-  </gazebo>
+  </gazebo> -->
   <joint name="frame3_fl_to_gear_fl" type="revolute">
-    <parent link="gear_fl"/>
+    <parent link="base_link"/>
     <child  link="frame3_fl"/>
     <axis xyz="0 0 1"/>
-    <origin xyz="0 0.02 -0.08" rpy="0 0 0"/>
+    <origin xyz="0.23 0.195 -0.205" rpy="0 0 0"/>
     <limit lower="-3.1415" upper="3.1415" effort="30" velocity="10"/>
     <dybamics damping="10000.0" friction="10000.0" />
@@ -493,9 +493,8 @@
     <type>transmission_interface/SimpleTransmission</type>
     <joint name="frame3_fl_to_gear_fl">
-        <hardwareInterface>hardware_interface/VelocityJointInterface</hardwareInterface>
+        <hardwareInterface>hardware_interface/PositionJointInterface</hardwareInterface>
     </joint>
     <actuator name="frame3_fl_to_gear_fl_motor">
-      <hardwareInterface>hardware_interface/VelocityJointInterface</hardwareInterface>
-      <mechanismReduction>1</mechanismReduction>
+      <hardwareInterface>hardware_interface/PositionJointInterface</hardwareInterface>
     </actuator>
   </transmission>
@@ -534,5 +533,5 @@
     <mu2 value="2500" />
   </gazebo>
-  <joint name="motor_fl_to_frame3_fl" type="fixed">
+  <!-- <joint name="motor_fl_to_frame3_fl" type="fixed">
     <parent link="frame3_fl"/>
     <child  link="motor_fl"/>
@@ -560,9 +559,9 @@
   <gazebo reference="motor_fl">
     <material>Gazebo/Grey</material>
-  </gazebo>
+  </gazebo> -->
   <joint name="wheel_fl_to_motor_fl" type="continuous">
-    <parent link="motor_fl"/>
+    <parent link="frame3_fl"/>
     <child  link="wheel_fl"/>
-    <origin xyz="0 0.09 0" rpy="0 0 0"/>
+    <origin xyz="0 0.02 -0.09" rpy="0 0 0"/>
     <!-- <origin xyz="0 0.15 0" rpy="0 0 0"/> -->
     <axis xyz="0 1 0"/>
@@ -576,7 +575,5 @@
     </joint>
     <actuator name="wheel_fl_motor">
-      <!-- <hardwareInterface>hardware_interface/VelocityJointInterface</hardwareInterface> -->
-      <hardwareInterface>EffortJointInterface</hardwareInterface>
-      <mechanismReduction>1</mechanismReduction>
+      <hardwareInterface>hardware_interface/VelocityJointInterface</hardwareInterface>
     </actuator>
   </transmission>
@@ -609,6 +606,50 @@
     <kd value="1.0" />
   </gazebo>
+   <!-- virtual steer -->
+  <joint name="front_steer_joint" type="revolute">
+    <parent link="base_link"/>
+    <child link="front_steer_link"/>
+    <axis xyz="0 0 1"/>
+    <origin xyz="0.23 0.093 -0.205" rpy="0 0 0"/>
+    <limit lower="-3.1415" upper="3.1415" effort="30" velocity="10"/>
+    <dybamics damping="10000.0" friction="10000.0" />
+  </joint>
+  <transmission name="front_steer_trans">
+    <type>transmission_interface/SimpleTransmission</type>
+    <joint name="front_steer_joint">
+        <hardwareInterface>hardware_interface/PositionJointInterface</hardwareInterface>
+    </joint>
+    <actuator name="front_steer_joint_motor">
+      <hardwareInterface>hardware_interface/PositionJointInterface</hardwareInterface>
+      <hardwareInterface>EffortJointInterface</hardwareInterface>
+      <mechanismReduction>1</mechanismReduction>
+    </actuator>
+  </transmission>
+  <link name="front_steer_link">
+    <visual>
+      <geometry>
+        <box size="0.075 0.09 0.09"/>
+      </geometry>
+      <origin xyz="0 0 0" rpy="0 0 0"/>
+      <material name="frame"/>
+    </visual>
+    <collision>
+      <geometry>
+        <box size="0.075 0.09 0.09"/>
+      </geometry>
+      <origin xyz="0 0 0" rpy="0 0 0"/>
+      <material name="frame"/>
+    </collision>
+    <inertial>
+      <origin xyz="0 0 0" rpy="0 0 0"/>
+      <mass value="1.0"/>
+      <inertia ixx="1.0" ixy="0.0" ixz="0.0" iyy="1.0" iyz="0.0" izz="1.0"/>
+    </inertial>
+  </link>
+    <gazebo reference="front_steer_joint">
+      <provideFeedback>true</provideFeedback>
+    </gazebo>
       <!-- leg_bl : mirror leg_fl to the y axis -->
-  <joint name="frame1_bl_to_base_link" type="fixed">
+  <!-- <joint name="frame1_bl_to_base_link" type="fixed">
     <parent link="base_link"/>
     <child  link="frame1_bl"/>
@@ -686,23 +727,23 @@
   <gazebo reference="gear_bl">
     <material>Gazebo/Blue</material>
-  </gazebo>
-  <joint name="frame3_bl_to_gear_bl" type="revolute">
-    <parent link="gear_bl"/>
+  </gazebo> -->
+  <joint name="frame3_bl_to_gear_bl" type="fixed">
+    <parent link="base_link"/>
     <child  link="frame3_bl"/>
     <axis xyz="0 0 1"/>
-    <origin xyz="0 0.02 -0.08" rpy="0 0 0"/>
-    <limit lower="-3.1415" upper="3.1415" effort="30" velocity="10"/>
-    <dybamics damping="10000.0" friction="10000.0" />
-  </joint>
-  <transmission name="frame3_bl_to_gear_bl_trans">
+    <origin xyz="-0.23 0.175 -0.205" rpy="0 0 0"/>
+    <!-- <limit lower="-3.1415" upper="3.1415" effort="30" velocity="10"/>
+    <dybamics damping="10000.0" friction="10000.0" /> -->
+  </joint>
+  <!-- <transmission name="frame3_bl_to_gear_bl_trans">
     <type>transmission_interface/SimpleTransmission</type>
     <joint name="frame3_bl_to_gear_bl">
-        <hardwareInterface>hardware_interface/VelocityJointInterface</hardwareInterface>
+        <hardwareInterface>hardware_interface/PositionJointInterface</hardwareInterface>
     </joint>
     <actuator name="frame3_bl_to_gear_bl_motor">
-      <hardwareInterface>hardware_interface/VelocityJointInterface</hardwareInterface>
+      <hardwareInterface>hardware_interface/PositionJointInterface</hardwareInterface>
       <mechanismReduction>1</mechanismReduction>
     </actuator>
-  </transmission>
+  </transmission> -->
   <!--<joint name="frame3_bl_to_gear_bl" type="fixed">
     <parent link="gear_bl"/>
@@ -736,5 +777,5 @@
     <mu2 value="2500" />
   </gazebo>
-  <joint name="motor_bl_to_frame3_bl" type="fixed">
+  <!-- <joint name="motor_bl_to_frame3_bl" type="fixed">
     <parent link="frame3_bl"/>
     <child  link="motor_bl"/>
@@ -762,9 +803,9 @@
   <gazebo reference="motor_bl">
     <material>Gazebo/Grey</material>
-  </gazebo>
+  </gazebo> -->
   <joint name="wheel_bl_to_motor_bl" type="continuous">
-    <parent link="motor_bl"/>
+    <parent link="base_link"/>
     <child  link="wheel_bl"/>
-    <origin xyz="0 0.09 0" rpy="0 0 0"/>
+    <origin xyz="-0.23 0.175 -0.295" rpy="0 0 0"/>
     <!-- <origin xyz="0 0.15 0" rpy="0 0 0"/> -->
     <axis xyz="0 1 0"/>
@@ -778,5 +819,5 @@
     </joint>
     <actuator name="wheel_bl_motor">
-      <!-- <hardwareInterface>hardware_interface/VelocityJointInterface</hardwareInterface> -->
+      <hardwareInterface>hardware_interface/VelocityJointInterface</hardwareInterface>
       <hardwareInterface>EffortJointInterface</hardwareInterface>
       <mechanismReduction>1</mechanismReduction>
@@ -812,5 +853,5 @@
   </gazebo>
     <!-- leg_fr -->
-  <joint name="frame1_fr_to_base_link" type="fixed">
+  <!-- <joint name="frame1_fr_to_base_link" type="fixed">
     <parent link="base_link"/>
     <child  link="frame1_fr"/>
@@ -888,10 +929,10 @@
   <gazebo reference="gear_fr">
     <material>Gazebo/Blue</material>
-  </gazebo>
+  </gazebo> -->
   <joint name="frame3_fr_to_gear_fr" type="revolute">
-    <parent link="gear_fr"/>
+    <parent link="base_link"/>
     <child  link="frame3_fr"/>
     <axis xyz="0 0 1"/>
-    <origin xyz="0 0.02 -0.08" rpy="0 0 0"/>
+    <origin xyz="0.23 -0.195 -0.205" rpy="0 0 0"/>
     <limit lower="-3.1415" upper="3.1415" effort="30" velocity="10"/>
     <dybamics damping="10000.0" friction="10000.0" />
@@ -900,8 +941,8 @@
     <type>transmission_interface/SimpleTransmission</type>
     <joint name="frame3_fr_to_gear_fr">
-        <hardwareInterface>hardware_interface/VelocityJointInterface</hardwareInterface>
+        <hardwareInterface>hardware_interface/PositionJointInterface</hardwareInterface>
     </joint>
     <actuator name="frame3_fr_to_gear_fr_motor">
-      <hardwareInterface>hardware_interface/VelocityJointInterface</hardwareInterface>
+      <hardwareInterface>hardware_interface/PositionJointInterface</hardwareInterface>
       <mechanismReduction>1</mechanismReduction>
     </actuator>
@@ -938,5 +979,5 @@
     <mu2 value="2500" />
   </gazebo>
-  <joint name="motor_fr_to_frame3_fr" type="fixed">
+  <!-- <joint name="motor_fr_to_frame3_fr" type="fixed">
     <parent link="frame3_fr"/>
     <child  link="motor_fr"/>
@@ -964,9 +1005,9 @@
   <gazebo reference="motor_fr">
     <material>Gazebo/Grey</material>
-  </gazebo>
+  </gazebo> -->
   <joint name="wheel_fr_to_motor_fr" type="continuous">
-    <parent link="motor_fr"/>
+    <parent link="frame3_fr"/>
     <child  link="wheel_fr"/>
-    <origin xyz="0 -0.09 0" rpy="0 0 0"/>
+    <origin xyz="0 0.02 -0.09" rpy="0 0 0"/>
    <!-- <origin xyz="0 -0.15 0" rpy="0 0 0"/>  -->
     <axis xyz="0 1 0"/>
@@ -980,5 +1021,5 @@
     </joint>
     <actuator name="wheel_fr_motor">
-      <!-- <hardwareInterface>hardware_interface/VelocityJointInterface</hardwareInterface> -->
+      <hardwareInterface>hardware_interface/VelocityJointInterface</hardwareInterface>
       <hardwareInterface>EffortJointInterface</hardwareInterface>
       <mechanismReduction>1</mechanismReduction>
@@ -1014,5 +1055,5 @@
   </gazebo>
     <!-- leg_br -->
-  <joint name="frame1_br_to_base_link" type="fixed">
+  <!-- <joint name="frame1_br_to_base_link" type="fixed">
     <parent link="base_link"/>
     <child  link="frame1_br"/>
@@ -1090,23 +1131,23 @@
   <gazebo reference="gear_br">
     <material>Gazebo/Blue</material>
-  </gazebo>
-  <joint name="frame3_br_to_gear_br" type="revolute">
-    <parent link="gear_br"/>
+  </gazebo> -->
+  <joint name="frame3_br_to_gear_br" type="fixed">
+    <parent link="base_link"/>
     <child  link="frame3_br"/>
     <axis xyz="0 0 1"/>
-    <origin xyz="0 0.02 -0.08" rpy="0 0 0"/>
-    <limit lower="-3.1415" upper="3.1415" effort="30" velocity="10"/>
-    <dybamics damping="10000.0" friction="10000.0" />
-  </joint>
-  <transmission name="frame3_br_to_gear_br_trans">
+    <origin xyz="-0.23 -0.195 -0.205" rpy="0 0 0"/>
+    <!-- <limit lower="-3.1415" upper="3.1415" effort="30" velocity="10"/>
+    <dybamics damping="10000.0" friction="10000.0" /> -->
+  </joint>
+  <!-- <transmission name="frame3_br_to_gear_br_trans">
     <type>transmission_interface/SimpleTransmission</type>
     <joint name="frame3_br_to_gear_br">
-        <hardwareInterface>hardware_interface/VelocityJointInterface</hardwareInterface>
+        <hardwareInterface>hardware_interface/PositionJointInterface</hardwareInterface>
     </joint>
     <actuator name="frame3_br_to_gear_br_motor">
-      <hardwareInterface>hardware_interface/VelocityJointInterface</hardwareInterface>
+      <hardwareInterface>hardware_interface/PositionJointInterface</hardwareInterface>
       <mechanismReduction>1</mechanismReduction>
     </actuator>
-  </transmission>
+  </transmission> -->
   <!--<joint name="frame3_br_to_gear_br" type="fixed">
     <parent link="gear_br"/>
@@ -1140,5 +1181,5 @@
     <mu2 value="2500" />
   </gazebo>
-  <joint name="motor_br_to_frame3_br" type="fixed">
+  <!-- <joint name="motor_br_to_frame3_br" type="fixed">
     <parent link="frame3_br"/>
     <child  link="motor_br"/>
@@ -1166,9 +1207,9 @@
   <gazebo reference="motor_br">
     <material>Gazebo/Grey</material>
-  </gazebo>
+  </gazebo> -->
   <joint name="wheel_br_to_motor_br" type="continuous">
-    <parent link="motor_br"/>
+    <parent link="base_link"/>
     <child  link="wheel_br"/>
-    <origin xyz="0 -0.09 0" rpy="0 0 0"/>
+    <origin xyz="-0.23 -0.175 -0.295" rpy="0 0 0"/>
     <!-- <origin xyz="0 -0.15 0" rpy="0 0 0"/> -->
     <axis xyz="0 1 0"/>
@@ -1182,5 +1223,5 @@
     </joint>
     <actuator name="wheel_br_motor">
-      <!-- <hardwareInterface>hardware_interface/VelocityJointInterface</hardwareInterface> -->
+      <hardwareInterface>hardware_interface/VelocityJointInterface</hardwareInterface>
       <hardwareInterface>EffortJointInterface</hardwareInterface>
       <mechanismReduction>1</mechanismReduction>
@@ -1215,37 +1256,51 @@
     <kd value="1.0" />
   </gazebo>
+ <!-- virtual wheel -->
+  <joint name="rear_wheel_joint" type="continuous">
+    <parent link="base_link"/>
+    <child  link="rear_wheel_link"/>
+    <origin xyz="-0.23 0.0 -0.295" rpy="0 0 0"/>
+    <!-- <origin xyz="0 -0.15 0" rpy="0 0 0"/> -->
+    <axis xyz="0 1 0"/>
+    <limit effort="100" velocity="100"/>
+    <dynamics damping="0.1" friction="0.0"/>
+  </joint>
+  <transmission name="rear_wheel_trans">
+    <type>transmission_interface/SimpleTransmission</type>
+    <joint name="rear_wheel_joint">
+        <hardwareInterface>hardware_interface/VelocityJointInterface</hardwareInterface>
+    </joint>
+    <actuator name="rear_wheel_joint_motor">
+      <hardwareInterface>hardware_interface/VelocityJointInterface</hardwareInterface>
+      <hardwareInterface>EffortJointInterface</hardwareInterface>
+      <mechanismReduction>1</mechanismReduction>
+    </actuator>
+  </transmission>
+  <link name="rear_wheel_link">
+  <visual>
+      <geometry>
+        <cylinder length="0.09" radius="0.1"/>
+      </geometry>
+      <origin xyz="0 0 0" rpy="1.57 0 0"/>
+      <material name="wheel"/>
+    </visual>
+    <collision>
+      <geometry>
+        <cylinder length="0.09" radius="0.1"/>
+      </geometry>
+      <origin xyz="0 0 0" rpy="1.57 0 0"/>
+      <material name="wheel"/>
+    </collision>
+    <inertial>
+      <origin xyz="0 0 0" rpy="0 0 0"/>
+      <mass value="1.0"/>
+      <inertia ixx="1.0" ixy="0.0" ixz="0.0" iyy="1.0" iyz="0.0" izz="1.0"/>
+    </inertial>
+  </link>
   <gazebo>
     <plugin name="gazebo_ros_control" filename="libgazebo_ros_control.so">
-      <!-- <robotNamespace>/pf1</robotNamespace>
-      <robotSimType>gazebo_ros_control/DefaultRobotHWSim</robotSimType>
-      <legacyModeNS>true</legacyModeNS> -->
-      <!-- <commandTopic>cmd_vel</commandTopic>
-      <odometryTopic>odom</odometryTopic>
-      <odometryFrame>odom</odometryFrame>
-      <leftJoint>wheel_left_joint</leftJoint>
-      <rightJoint>wheel_right_joint</rightJoint> -->
+    <robotSimType>steer_bot_hardware_gazebo/SteerBotHardwareGazebo</robotSimType>
+    <legacyModeNS>false</legacyModeNS>
     </plugin>
   </gazebo>
-  <!-- <gazebo>
-    <plugin name="gazebo_ros_control" filename="libgazebo_ros_control.so">
-      <commandTopic>cmd_vel</commandTopic>
-      <odometryTopic>odom</odometryTopic>
-      <odometryFrame>odom</odometryFrame>
-      <odometrySource>world</odometrySource>
-      <publishOdomTF>true</publishOdomTF>
-      <robotBaseFrame>base_footprint</robotBaseFrame>
-      <publishWheelTF>false</publishWheelTF>
-      <publishTf>true</publishTf>
-      <publishWheelJointState>true</publishWheelJointState>
-      <legacyMode>true</legacyMode>
-      <updateRate>30</updateRate>
-      <leftJoint>wheel_left_joint</leftJoint>
-      <rightJoint>wheel_right_joint</rightJoint>
-      <wheelSeparation>0.160</wheelSeparation>
-      <wheelDiameter>0.066</wheelDiameter>
-      <wheelAcceleration>1</wheelAcceleration>
-      <wheelTorque>10</wheelTorque>
-      <rosDebugLevel>na</rosDebugLevel>
-    </plugin>
-  </gazebo> -->
 </robot>
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