Commit message: マッピングの追加

File: cdc_navigation/xacro/pf1.xacro (robot description, xacro)
@@ -24,7 +24,7 @@
   </material>
     <!-- base_footprint-->
-  <!-- <link name="base_footprint"/>
-  <gazebo reference="body_footprint"/>
-  <joint name="base_joint" type="fixed">
+  <!-- <link name="base_footprint"/> -->
+  <!-- <gazebo reference="body_footprint"/> -->
+  <!-- <joint name="base_joint" type="fixed">
     <parent link="base_footprint"/>
     <child link="base_link"/>
