Commit message: 追従のアルゴリズムを導入、検証済み→見失い時の処理系なし

File: cdc_navigation/xacro/PF1_stl.xacro (robot description, xacro)
@@ -23,8 +23,11 @@
     <color rgba="0.15 0.15 0.15 1.0"/>
   </material>
+  <material name="yellow">
+        <color rgba="0.8 0.8 0 1"/>
+  </material>
     <!-- base_footprint-->
-  <!-- <link name="base_footprint"/> -->
-  <!-- <gazebo reference="body_footprint"/> -->
-  <!-- <joint name="base_joint" type="fixed">
+  <!-- <link name="base_footprint"/>
+  <gazebo reference="body_footprint"/>
+  <joint name="base_joint" type="fixed">
     <parent link="base_footprint"/>
     <child link="base_link"/>
@@ -34,26 +37,41 @@
   <link name="base_link">
     <inertial>
-      <origin xyz="0 0 0" rpy="0 0 0"/>
+      <origin xyz="0 0 0.15" rpy="0 0 0"/>
       <mass value="10.0"/>
       <inertia ixx="1.0" ixy="0.0" ixz="0.0" iyy="1.0" iyz="0.0" izz="1.0"/>
     </inertial>
     <visual>
-      <geometry>
-        <box size="0.45 0.39 0.2"/>
-      </geometry>
-      <origin xyz="0 0 0" rpy="0 0 0"/>
-      <material name="base_link"/>
-    </visual>
-    <collision>
-      <geometry>
-        <box size="0.45 0.39 0.2"/>
-      </geometry>
-      <origin xyz="0 0 0" rpy="0 0 0"/>
-      <material name="base_link"/>
-    </collision>
-  </link>
-  <gazebo reference="body_link">
-    <material>Gazebo/White</material>
-  </gazebo>
+      <origin xyz="0 0 -0.05" rpy="0 0 0"/>
+      <geometry>
+        <mesh filename="package://cdc_navigation/meshes/pf1_body_ros_new.stl"/>
+      </geometry>
+    </visual>
+    <collision>
+      <geometry>
+        <mesh filename="package://cdc_navigation/meshes/pf1_body_ros_new.stl"/>
+      </geometry>
+    </collision>
+  </link>
+  <gazebo reference="base_link">
+    <!-- <material>Gazebo/White</material> -->
+    <material>Gazebo/Grey</material>
+  </gazebo>
+  <!-- <link name="base_link">
+    <visual>
+      <geometry>
+        <mesh filename="package://cdc_navigation/meshes/pf1_body_ros.dae"/>
+      </geometry>
+    </visual>
+    <collision>
+      <geometry>
+        <mesh filename="package://cdc_navigation/meshes/pf1_body_ros.dae"/>
+      </geometry>
+    </collision>
+    <inertial>
+      <origin rpy="0 0 0" xyz="-0.013 0 0"/>
+      <mass value="0.5"/>
+      <inertia ixx="0.00144" ixy="-0.000003703103" ixz="0.000005540558" iyy="0.0008207" iyz="0.000000571374" izz="0.001299"/>
+    </inertial>
+  </link> -->
     <!-- imu_link -->
   <joint name="imu_link_to_base_link" type="fixed">
@@ -99,8 +117,8 @@
   </gazebo>
     <!-- base_sensor -->
-  <joint name="base_link_to_base_sensor" type="fixed">
+  <!-- <joint name="base_link_to_base_sensor" type="fixed">
     <parent link="base_link"/>
     <child link="base_sensor"/>
-    <origin xyz="-0 0 0" rpy="0 0 0"/>
+    <origin xyz="0 0 0.28" rpy="0 0 0"/>
   </joint>
   <link name="base_sensor">
@@ -108,7 +126,6 @@
       <origin xyz="0 0 0.0" rpy="0 0 0"/>
       <geometry>
-        <cylinder length="0.01" radius="0.005"/>
-      </geometry>
-      <material name="lidar"/>
+        <mesh filename="package://rrbot_description/meshes/hokuyo.dae"/>
+      </geometry>
     </visual>
     <collision>
@@ -122,5 +139,61 @@
   <gazebo reference="base_link_to_base_sensor">
     <material>Gazebo/Grey</material>
-  </gazebo>
+  </gazebo> -->
+  <joint name="hokuyo_joint" type="fixed">
+      <parent link="base_link"/>
+      <child  link="hokuyo_sensor"/>
+      <!-- <origin xyz="0.02 0 0.27" rpy="0 0 0"/> -->
+      <origin xyz="0.18 0 0.27" rpy="0 0 0"/>
+    </joint>
+<link name="hokuyo_sensor">
+   <collision>
+      <origin xyz="0 0 0.3" rpy="0 0 0"/>
+      <geometry>
+        <box size="0.1 0.1 0.1"/>
+      </geometry>
+    </collision>
+    <visual>
+      <origin xyz="0 0 -0.1" rpy="0 0 0"/>
+      <geometry>
+        <mesh filename="package://rrbot_description/meshes/hokuyo.dae"/>
+      </geometry>
+    </visual>
+    <inertial>
+      <mass value="1e-5" />
+      <origin xyz="0 0 0" rpy="0 0 0"/>
+      <inertia ixx="1e-6" ixy="0" ixz="0" iyy="1e-6" iyz="0" izz="1e-6" />
+    </inertial>
+    </link>
+    <gazebo reference="hokuyo_sensor">
+      <sensor type="ray" name="base_link_hokuyo_sensor">
+        <pose>0 0 0 0 0 0</pose>
+        <visualize>false</visualize>
+        <update_rate>40</update_rate>
+        <ray>
+          <scan>
+            <horizontal>
+                <samples>400</samples>
+                <resolution>1</resolution>
+                <min_angle>${radians(-180)}</min_angle>
+                <max_angle>${radians( 180)}</max_angle>
+            </horizontal>
+          </scan>
+          <range>
+            <min>0.10</min>
+            <max>30.0</max>
+            <resolution>0.01</resolution>
+          </range>
+          <noise>
+            <type>gaussian</type>
+            <mean>0.0</mean>
+            <stddev>0.01</stddev>
+          </noise>
+        </ray>
+        <plugin name="gazebo_ros_lidar_controller" filename="libgazebo_ros_laser.so">
+          <topicName>scan</topicName>
+          <frameName>hokuyo_sensor</frameName>
+        </plugin>
+      </sensor>
+    </gazebo>
     <!-- realsense -->
   <!-- set property -->
@@ -137,10 +210,11 @@
     <joint name="camera_joint" type="fixed">
       <origin xyz="0.225 0 0" rpy="0 0 0" />
-      <parent link="base_sensor" />
+      <!-- <parent link="base_sensor" /> -->
+      <parent link="base_link" />
       <child link="camera_bottom_screw_frame" />
     </joint>
     <link name="camera_bottom_screw_frame"/>
     <joint name="camera_link_joint" type="fixed">
-      <origin xyz="0.0125 0 0" rpy="0 0 0"/>
+      <origin xyz="0.01 0.018 0.1" rpy="0 0 0"/>
       <!--<origin xyz="0.08 ${d435_cam_depth_py} 0.055" rpy="0 0 0"/>-->
       <parent link="camera_bottom_screw_frame"/>
@@ -149,5 +223,5 @@
     <link name="camera_link">
       <visual>
-        <origin xyz="0 ${-d435_cam_depth_py} 0" rpy="${M_PI/2} 0 ${M_PI/2}"/>
+        <origin xyz="-0.02 ${-d435_cam_depth_py} 0" rpy="${M_PI/2} 0 ${M_PI/2}"/>
         <geometry>
           <box size="${d435_cam_width} ${d435_cam_height} ${d435_cam_depth}" />
@@ -255,13 +329,5 @@
             <width>1280</width>
             <height>720</height>
-          </image>
-          <clip>
-            <near>0.1</near>
-            <far>1000</far>
-          </clip>
-          <noise>
-            <type>gaussian</type>
-            <mean>0.0</mean>
-            <stddev>0.100</stddev>
+          </image><!--end of realsense setup-->
           </noise>
         </camera>
@@ -342,5 +408,5 @@
         <infrared2OpticalframeName>infrared2_optical_frame</infrared2OpticalframeName>
         <rangeMinDepth>0.2</rangeMinDepth>
-        <rangeMaxDepth>400.0</rangeMaxDepth>
+        <rangeMaxDepth>10.0</rangeMaxDepth>
         <pointCloud>true</pointCloud>
         <pointCloudTopicName>depth/color/points</pointCloudTopicName>
@@ -349,142 +415,9 @@
       </plugin>
     </gazebo>
-    <!--end of realsense setup-->
-     <link name="hokuyo_sensor">
-   <collision>
-      <origin xyz="0 0 0" rpy="0 0 0"/>
-      <geometry>
-        <box size="0.1 0.1 0.1"/>
-      </geometry>
-    </collision>
-    <visual>
-      <origin xyz="0 0 0" rpy="0 0 0"/>
-      <geometry>
-        <mesh filename="package://rrbot_description/meshes/hokuyo.dae"/>
-      </geometry>
-    </visual>
-    <inertial>
-      <mass value="1e-5" />
-      <origin xyz="0 0 0" rpy="0 0 0"/>
-      <inertia ixx="1e-6" ixy="0" ixz="0" iyy="1e-6" iyz="0" izz="1e-6" />
-    </inertial>
-    </link>
-    <joint name="hokuyo_joint" type="fixed">
-      <parent link="base_link"/>
-      <child  link="hokuyo_sensor"/>
-      <origin xyz="0.02 0 0.13" rpy="0 0 0"/>
-    </joint>
-    <gazebo reference="hokuyo_sensor">
-      <sensor type="ray" name="base_link_hokuyo_sensor">
-        <pose>0 0 0 0 0 0</pose>
-        <visualize>false</visualize>
-        <update_rate>40</update_rate>
-        <ray>
-          <scan>
-          <horizontal>
-                <samples>400</samples>
-                <resolution>1</resolution>
-                <min_angle>${radians(-180)}</min_angle>
-                <max_angle>${radians( 180)}</max_angle>
-          </horizontal>
-          </scan>
-          <range>
-            <min>0.10</min>
-            <max>30.0</max>
-            <resolution>0.01</resolution>
-          </range>
-          <noise>
-            <type>gaussian</type>
-            <stddev>0.01</stddev>
-          </noise>
-        </ray>
-        <plugin name="gazebo_ros_lidar_controller" filename="libgazebo_ros_laser.so">
-          <topicName>scan</topicName>
-          <frameName>hokuyo_sensor</frameName>
-        </plugin>
-      </sensor>
-    </gazebo>
-    <!-- leg_fl -->
-  <!-- <joint name="frame1_fl_to_base_link" type="fixed">
-    <parent link="base_link"/>
-    <child  link="frame1_fl"/>
-    <origin xyz="0 0.14 -0.1" rpy="0 0 0"/>
-  </joint>
-  <link name="frame1_fl">
-    <visual>
-      <geometry>
-        <box size="0.27 0.02 0.09"/>
-      </geometry>
-      <origin xyz="0.135 0 0" rpy="0 0 0"/>
-      <material name="frame"/>
-    </visual>
-    <collision>
-      <geometry>
-        <box size="0.27 0.02 0.09"/>
-      </geometry>
-      <origin xyz="0.135 0 0" rpy="0 0 0"/>
-      <material name="frame"/>
-    </collision>
-  </link>
-  <gazebo reference="frame1_fl">
-    <material>Gazebo/Grey</material>
-  </gazebo>
-  <joint name="frame2_fl_to_frame1_fl" type="fixed">
-    <parent link="frame1_fl"/>
-    <child  link="frame2_fl"/>
-    <origin xyz="0.23 0.02 -0.045" rpy="0 0 0"/>
-  </joint>
-  <link name="frame2_fl">
-    <visual>
-      <geometry>
-        <box size="0.08 0.02 0.05"/>
-      </geometry>
-      <origin xyz="0 0 0" rpy="0 0 0"/>
-      <material name="frame"/>
-    </visual>
-    <collision>
-      <geometry>
-        <box size="0.08 0.02 0.05"/>
-      </geometry>
-      <origin xyz="0 0 0" rpy="0 0 0"/>
-      <material name="frame"/>
-    </collision>
-  </link>
-  <gazebo reference="frame2_fl">
-    <material>Gazebo/Grey</material>
-  </gazebo>
-  <joint name="gear_fl_to_frame2_fl" type="fixed">
-    <parent link="frame2_fl"/>
-    <child  link="gear_fl"/>
-    <origin xyz="0 0.035 -0.06" rpy="0 0 0"/>
-  </joint>
-  <link name="gear_fl">
-    <visual>
-      <geometry>
-        <box size="0.075 0.09 0.07"/>
-      </geometry>
-      <origin xyz="0 0 0" rpy="0 0 0"/>
-      <material name="gear"/>
-    </visual>
-    <collision>
-      <geometry>
-        <box size="0.075 0.09 0.07"/>
-      </geometry>
-      <origin xyz="0 0 0" rpy="0 0 0"/>
-      <material name="gear"/>
-    </collision>
-    <inertial>
-      <origin xyz="0 0 0" rpy="0 0 0"/>
-      <mass value="1.0"/>
-      <inertia ixx="1.0" ixy="0.0" ixz="0.0" iyy="1.0" iyz="0.0" izz="1.0"/>
-    </inertial>
-  </link>
-  <gazebo reference="gear_fl">
-    <material>Gazebo/Blue</material>
-  </gazebo> -->
   <joint name="frame3_fl_to_gear_fl" type="revolute">
     <parent link="base_link"/>
     <child  link="frame3_fl"/>
     <axis xyz="0 0 1"/>
-    <origin xyz="0.23 0.195 -0.205" rpy="0 0 0"/>
+    <origin xyz="0.165 0.125 -0.31" rpy="0 0 0"/>
     <limit lower="-3.1415" upper="3.1415" effort="30" velocity="10"/>
     <dybamics damping="10000.0" friction="10000.0" />
@@ -499,26 +432,15 @@
     </actuator>
   </transmission>
-  <!-- <gazebo reference="frame3_fl_to_gear_fl">
-    <material>Gazebo/Blue</material>
-  </gazebo> -->
-  <!--<joint name="frame3_fl_to_gear_fl" type="fixed">
-    <parent link="gear_fl"/>
-    <child  link="frame3_fl"/>
-    <origin xyz="0 0.0 -0.08" rpy="0 0 0"/>
-  </joint>-->
   <link name="frame3_fl">
     <visual>
-      <geometry>
-        <box size="0.075 0.09 0.09"/>
-      </geometry>
-      <origin xyz="0 0 0" rpy="0 0 0"/>
-      <material name="frame"/>
-    </visual>
-    <collision>
-      <geometry>
-        <box size="0.075 0.09 0.09"/>
-      </geometry>
-      <origin xyz="0 0 0" rpy="0 0 0"/>
-      <material name="frame"/>
+      <origin xyz="0 0 0" rpy="0 0 0"/>
+      <geometry>
+        <mesh filename="package://cdc_navigation/meshes/pf1_steer_only_zero_ros.stl"/>
+      </geometry>
+    </visual>
+    <collision>
+      <geometry>
+        <mesh filename="package://cdc_navigation/meshes/pf1_steer_only_zero_ros.stl"/>
+      </geometry>
     </collision>
     <inertial>
@@ -533,35 +455,10 @@
     <mu2 value="2500" />
   </gazebo>
-  <!-- <joint name="motor_fl_to_frame3_fl" type="fixed">
-    <parent link="frame3_fl"/>
-    <child  link="motor_fl"/>
-    <origin xyz="0 -0.02 -0.09" rpy="0 0 0"/>
-  </joint>
-  <link name="motor_fl">
-    <visual>
-      <geometry>
-        <box size="0.075 0.09 0.09"/>
-      </geometry>
-      <material name="motor"/>
-    </visual>
-    <collision>
-      <geometry>
-        <box size="0.075 0.09 0.09"/>
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